File: RobotSuiveurDeLigne/RobotSuiveurDeLigne.kicad_sch (KiCad schematic)
At the start: 22 parts, among them J1 US_IUT_VdA, J2 Conn_02x05_Odd_Even, U1 CNY70_IUT_VdA, U2 CNY70_IUT_VdA, U3 CNY70_IUT_VdA, U4 CNY70_IUT_VdA, U5 CNY70_IUT_VdA, U6 CNY70_IUT_VdA

Commit message: modifs shéma
Other:
- company: (none) -> IUT de Ville d'Avray
- title: (none) -> CAO - Robot Suiveur de Ligne
Changed lines of the file:
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@@
 	(generator_version "8.0")
 	(paper "A4")
+	(title_block
+		(title "CAO - Robot Suiveur de Ligne")
+		(company "IUT de Ville d'Avray")
+		(comment 1 "Gabriel PORTIER")
+		(comment 2 "Alexandre POPESCU")
+		(comment 3 "TP6")
+	)
 	(junction
 		(at 195.58 29.21)
@@
 	)
 	(junction
+		(at 100.33 107.95)
+		(diameter 0)
+		(color 0 0 0 0)
+	)
+	(junction
 		(at 190.5 57.15)
 		(diameter 0)
@@
 	)
 	(junction
+		(at 101.6 96.52)
+		(diameter 0)
+		(color 0 0 0 0)
+	)
+	(junction
 		(at 127 44.45)
 		(diameter 0)
@@
 	(wire
 		(pts
-			(xy 95.25 96.52) (xy 105.41 96.52)
+			(xy 95.25 96.52) (xy 101.6 96.52)
 		)
 		(stroke
@@
 	(wire
 		(pts
+			(xy 100.33 107.95) (xy 105.41 107.95)
+		)
+		(stroke
+			(width 0)
+			(type default)
+		)
+	)
+	(wire
+		(pts
 			(xy 92.71 44.45) (xy 92.71 48.26)
 		)
@@
 	(wire
 		(pts
+			(xy 101.6 96.52) (xy 105.41 96.52)
+		)
+		(stroke
+			(width 0)
+			(type default)
+		)
+	)
+	(wire
+		(pts
 			(xy 224.79 57.15) (xy 226.06 57.15)
 		)
@@
 	(wire
 		(pts
-			(xy 95.25 107.95) (xy 105.41 107.95)
+			(xy 95.25 107.95) (xy 100.33 107.95)
 		)
 		(stroke
@@
 	(wire
 		(pts
-			(xy 105.41 93.98) (xy 105.41 96.52)
+			(xy 101.6 90.17) (xy 101.6 96.52)
 		)
 		(stroke
@@
 	(wire
 		(pts
-			(xy 105.41 107.95) (xy 105.41 110.49)
+			(xy 100.33 107.95) (xy 100.33 118.11)
 		)
 		(stroke
@@
 	(symbol
 		(lib_id "power:PWR_FLAG")
-		(at 105.41 110.49 180)
+		(at 100.33 118.11 180)
 		(unit 1)
 		(exclude_from_sim no)
@@
 		(fields_autoplaced yes)
 		(property "Reference" "#FLG02"
-			(at 105.41 112.395 0)
+			(at 100.33 120.015 0)
 			(effects
 				(font
@@
 		)
 		(property "Value" "PWR_FLAG"
-			(at 105.41 115.57 0)
+			(at 100.33 123.19 0)
 			(effects
 				(font
@@
 		)
 		(property "Footprint" ""
-			(at 105.41 110.49 0)
+			(at 100.33 118.11 0)
 			(effects
 				(font
@@
 		)
 		(property "Datasheet" "~"
-			(at 105.41 110.49 0)
+			(at 100.33 118.11 0)
 			(effects
 				(font
@@
 		)
 		(property "Description" "Special symbol for telling ERC where power comes from"
-			(at 105.41 110.49 0)
+			(at 100.33 118.11 0)
 			(effects
 				(font
@@
 	(symbol
 		(lib_id "power:PWR_FLAG")
-		(at 105.41 93.98 0)
+		(at 101.6 90.17 0)
 		(unit 1)
 		(exclude_from_sim no)
@@
 		(fields_autoplaced yes)
 		(property "Reference" "#FLG01"
-			(at 105.41 92.075 0)
+			(at 101.6 88.265 0)
 			(effects
 				(font
@@
 		)
 		(property "Value" "PWR_FLAG"
-			(at 105.41 88.9 0)
+			(at 101.6 85.09 0)
 			(effects
 				(font
@@
 		)
 		(property "Footprint" ""
-			(at 105.41 93.98 0)
+			(at 101.6 90.17 0)
 			(effects
 				(font
@@
 		)
 		(property "Datasheet" "~"
-			(at 105.41 93.98 0)
+			(at 101.6 90.17 0)
 			(effects
 				(font
@@
 		)
 		(property "Description" "Special symbol for telling ERC where power comes from"
-			(at 105.41 93.98 0)
-			(effects
-				(font
+			(at 101.6 90.17 0)
+			(effects
+				(font

Commit message: ajout empreintes pour routage
Parts:
- C1: footprint (none) -> Capacitor_THT:CP_Radial_D13.0mm_P5.00mm
- C2: footprint (none) -> Capacitor_THT:CP_Radial_D6.3mm_P2.50mm
- J1: footprint (none) -> US:UltraSon_IUT_VdA
- J2: footprint (none) -> Connector_PinHeader_2.54mm:PinHeader_2x05_P2.54mm_Horizontal
- R1, R10, R11, R12, R2, R3, R4, R5, R6, R7, R8, R9: footprint (none) -> Resistor_THT:R_Axial_DIN0207_L6.3mm_D2.5mm_P10.16mm_Horizontal
- U1, U2, U3, U4, U5, U6: footprint (none) -> OptoDevice:Vishay_CNY70
Changed lines of the file:
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@@
 			)
 		)
-		(property "Footprint" ""
+		(property "Footprint" "Resistor_THT:R_Axial_DIN0207_L6.3mm_D2.5mm_P10.16mm_Horizontal"
 			(at 125.222 40.64 90)
 			(effects
@@
 			)
 		)
-		(property "Footprint" ""
+		(property "Footprint" "Resistor_THT:R_Axial_DIN0207_L6.3mm_D2.5mm_P10.16mm_Horizontal"
 			(at 201.422 40.64 90)
 			(effects
@@
 			)
 		)
-		(property "Footprint" ""
+		(property "Footprint" "OptoDevice:Vishay_CNY70"
 			(at 45.72 52.07 0)
 			(effects
@@
 			)
 		)
-		(property "Footprint" ""
+		(property "Footprint" "Resistor_THT:R_Axial_DIN0207_L6.3mm_D2.5mm_P10.16mm_Horizontal"
 			(at 56.642 40.64 90)
 			(effects
@@
 			)
 		)
-		(property "Footprint" ""
+		(property "Footprint" "Connector_PinHeader_2.54mm:PinHeader_2x05_P2.54mm_Horizontal"
 			(at 218.44 88.9 0)
 			(effects
@@
 			)
 		)
-		(property "Footprint" ""
+		(property "Footprint" "Resistor_THT:R_Axial_DIN0207_L6.3mm_D2.5mm_P10.16mm_Horizontal"
 			(at 193.802 40.64 90)
 			(effects
@@
 			)
 		)
-		(property "Footprint" ""
+		(property "Footprint" "Resistor_THT:R_Axial_DIN0207_L6.3mm_D2.5mm_P10.16mm_Horizontal"
 			(at 167.132 40.64 90)
 			(effects
@@
 			)
 		)
-		(property "Footprint" ""
+		(property "Footprint" "Resistor_THT:R_Axial_DIN0207_L6.3mm_D2.5mm_P10.16mm_Horizontal"
 			(at 98.552 40.64 90)
 			(effects
@@
 			)
 		)
-		(property "Footprint" ""
+		(property "Footprint" "Resistor_THT:R_Axial_DIN0207_L6.3mm_D2.5mm_P10.16mm_Horizontal"
 			(at 159.512 40.64 90)
 			(effects
@@
 			)
 		)
-		(property "Footprint" ""
+		(property "Footprint" "OptoDevice:Vishay_CNY70"
 			(at 114.3 52.07 0)
 			(effects
@@
 			)
 		)
-		(property "Footprint" ""
+		(property "Footprint" "Resistor_THT:R_Axial_DIN0207_L6.3mm_D2.5mm_P10.16mm_Horizontal"
 			(at 29.972 40.64 90)
 			(effects
@@
 			)
 		)
-		(property "Footprint" ""
+		(property "Footprint" "Resistor_THT:R_Axial_DIN0207_L6.3mm_D2.5mm_P10.16mm_Horizontal"
 			(at 228.092 40.64 90)
 			(effects
@@
 			)
 		)
-		(property "Footprint" ""
+		(property "Footprint" "OptoDevice:Vishay_CNY70"
 			(at 148.59 52.07 0)
 			(effects
@@
 			)
 		)
-		(property "Footprint" ""
+		(property "Footprint" "OptoDevice:Vishay_CNY70"
 			(at 80.01 52.07 0)
 			(effects
@@
 			)
 		)
-		(property "Footprint" ""
+		(property "Footprint" "Resistor_THT:R_Axial_DIN0207_L6.3mm_D2.5mm_P10.16mm_Horizontal"
 			(at 90.932 40.64 90)
 			(effects
@@
 			)
 		)
-		(property "Footprint" ""
+		(property "Footprint" "Resistor_THT:R_Axial_DIN0207_L6.3mm_D2.5mm_P10.16mm_Horizontal"
 			(at 132.842 40.64 90)
 			(effects
@@
 			)
 		)
-		(property "Footprint" ""
+		(property "Footprint" "Capacitor_THT:CP_Radial_D13.0mm_P5.00mm"
 			(at 106.3752 105.41 0)
 			(effects
@@
 			)
 		)
-		(property "Footprint" ""
+		(property "Footprint" "US:UltraSon_IUT_VdA"
 			(at 261.62 86.36 0)
 			(effects
@@
 			)
 		)
-		(property "Footprint" ""
+		(property "Footprint" "Capacitor_THT:CP_Radial_D6.3mm_P2.50mm"
 			(at 115.2652 105.41 0)
 			(effects
@@
 			)
 		)
-		(property "Footprint" ""
+		(property "Footprint" "Resistor_THT:R_Axial_DIN0207_L6.3mm_D2.5mm_P10.16mm_Horizontal"
 			(at 64.262 40.64 90)
 			(effects
@@
 			)
 		)
-		(property "Footprint" ""
+		(property "Footprint" "OptoDevice:Vishay_CNY70"
 			(at 217.17 52.07 0)
 			(effects
@@
 			)
 		)
-		(property "Footprint" ""
+		(property "Footprint" "OptoDevice:Vishay_CNY70"
 			(at 182.88 52.07 0)
 			(effects

Commit message: ajouts et changements mineurs
ajout condensateur + résistances
Parts:
- C1: footprint Capacitor_THT:CP_Radial_D13.0mm_P5.00mm -> Capacitor_THT:C_Rect_L7.0mm_W6.5mm_P5.00mm
- J2: footprint Connector_PinHeader_2.54mm:PinHeader_2x05_P2.54mm_Horizontal -> Connector_IDC:IDC-Header_2x05_P2.54mm_Horizontal
Changed lines of the file:
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@@
 			)
 		)
-		(property "Footprint" "Connector_PinHeader_2.54mm:PinHeader_2x05_P2.54mm_Horizontal"
+		(property "Footprint" "Connector_IDC:IDC-Header_2x05_P2.54mm_Horizontal"
 			(at 218.44 88.9 0)
 			(effects
@@
 			)
 		)
-		(property "Footprint" "Capacitor_THT:CP_Radial_D13.0mm_P5.00mm"
+		(property "Footprint" "Capacitor_THT:C_Rect_L7.0mm_W6.5mm_P5.00mm"
 			(at 106.3752 105.41 0)
 			(effects
