File: RobotSuiveurDeLigne/RobotSuiveurDeLigne.kicad_pcb (KiCad board)
At the start: 2 copper layers, 108 x 48 mm, 26 parts, among them J1 US_IUT_VdA, J2 Conn_02x05_Odd_Even, U1 CNY70_IUT_VdA, U2 CNY70_IUT_VdA, U3 CNY70_IUT_VdA, U4 CNY70_IUT_VdA, U5 CNY70_IUT_VdA, U6 CNY70_IUT_VdA

Commit message: Version alt du pcb v2.6
Parts:
- moved C1 0.50 mm to (113.0, 104.0)
- moved C2 0.50 mm to (122.0, 103.0)
Routing:
- net /D0: track 209.0 -> 230.1 mm, vias 1 -> 0
- net Net-(J2-Pin_4): track 128.0 -> 143.7 mm
- net VCC: track 215.9 -> 225.8 mm, vias 2 -> 1
- net /AN1: track 37.9 -> 28.0 mm
- net Net-(J2-Pin_2): track 127.9 -> 137.4 mm
- net /D1: track 88.6 -> 81.9 mm, vias 1 -> 0
- net Net-(U2-A): track 10.5 -> 11.4 mm
- net /AN0: track 20.8 -> 21.4 mm
- net Net-(U3-A): track 9.92 -> 10.5 mm

Commit message: Ajustement Vcc US
Continuité de la alt_v2.6
Routing:
- net VCC: track 225.8 -> 228.7 mm, vias 1 -> 2
- net Net-(J2-Pin_2): track 137.4 -> 136.7 mm
Changed lines of the file:
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@@
+	)
+	(segment
+		(start 140 63)
+		(end 132.5 63)
+		(width 0.4)
+		(layer "F.Cu")
+		(net 2)
 	)
 	(segment
@@
 		(width 0.4)
 		(layer "F.Cu")
+		(net 2)
+	)
+	(via
+		(at 132.5 63)
+		(size 2)
+		(drill 0.8)
+		(layers "F.Cu" "B.Cu")
 		(net 2)
 	)
@@
 	)
 	(segment
-		(start 130.5 70)
-		(end 137.5 63)
-		(width 0.4)
-		(layer "B.Cu")
-		(net 2)
-	)
-	(segment
-		(start 137.5 63)
-		(end 140 63)
-		(width 0.4)
-		(layer "B.Cu")
-		(net 2)
-	)
-	(segment
-		(start 133 62.5)
-		(end 136.5 66)
-		(width 0.4)
-		(layer "F.Cu")
-		(net 3)
+		(start 132.5 63)
+		(end 132.5 68)
+		(width 0.4)
+		(layer "B.Cu")
+		(net 2)
+	)
+	(segment
+		(start 132.5 68)
+		(end 130.5 70)
+		(width 0.4)
+		(layer "B.Cu")
+		(net 2)
 	)
 	(segment
@@
 	)
 	(segment
-		(start 96.2 62.5)
-		(end 133 62.5)
+		(start 126 62.5)
+		(end 129 65.5)
 		(width 0.4)
 		(layer "F.Cu")
@@
 	)
 	(segment
-		(start 136.5 66)
-		(end 141.5 66)
-		(width 0.4)
-		(layer "F.Cu")
-		(net 3)
-	)
-	(segment
-		(start 142.54 64.96)
-		(end 142.54 63)
+		(start 141.5 65.5)
+		(end 142.54 64.46)
+		(width 0.4)
+		(layer "F.Cu")
+		(net 3)
+	)
+	(segment
+		(start 96.2 62.5)
+		(end 126 62.5)
 		(width 0.4)
 		(layer "F.Cu")
@@
 	)
 	(segment
-		(start 141.5 66)
-		(end 142.54 64.96)
-		(width 0.4)
-		(layer "F.Cu")
-		(net 3)
-	)
-	(segment
 		(start 138.92 103.54)
 		(end 136.46 106)
@@
 	)
 	(segment
+		(start 129 65.5)
+		(end 141.5 65.5)
+		(width 0.4)
+		(layer "F.Cu")
+		(net 3)
+	)
+	(segment
+		(start 142.54 64.46)
+		(end 142.54 63)
+		(width 0.4)
+		(layer "F.Cu")
+		(net 3)
+	)
+	(segment
 		(start 121.2 60.8)
 		(end 144.3 60.8)
@@
 	)
 	(segment
-		(start 165 62)
-		(end 160.2 66.8)
-		(width 0.4)
-		(layer "F.Cu")
-		(net 7)
-	)
-	(segment
-		(start 160.2 66.8)
-		(end 135.8 66.8)
-		(width 0.4)
-		(layer "F.Cu")
-		(net 7)
-	)
-	(segment
 		(start 193.5 98.3)
 		(end 193.5 64)
@@
 	)
 	(segment
-		(start 105.5 74)
-		(end 107.5 72)
+		(start 95.3 64.7)
+		(end 96.5 63.5)
 		(width 0.4)
 		(layer "F.Cu")
@@
 	)
 	(segment
-		(start 135.8 66.8)
-		(end 132.5 63.5)
-		(width 0.4)
-		(layer "F.Cu")
-		(net 7)
-	)
-	(segment
-		(start 132.5 63.5)
-		(end 96.5 63.5)
-		(width 0.4)
-		(layer "F.Cu")
-		(net 7)
-	)
-	(segment
-		(start 96.3 74)
-		(end 105.5 74)
+		(start 107.5 70)
+		(end 107.5 72)
 		(width 0.4)
 		(layer "F.Cu")
@@
 	(segment
 		(start 96.5 63.5)
-		(end 95.3 64.7)
+		(end 125.868629 63.5)
+		(width 0.4)
+		(layer "F.Cu")
+		(net 7)
+	)
+	(segment
+		(start 125.868629 63.5)
+		(end 128.668629 66.3)
 		(width 0.4)
 		(layer "F.Cu")
@@
 	)
 	(segment
-		(start 95.3 73)
-		(end 96.3 74)
+		(start 160.7 66.3)
+		(end 165 62)
+		(width 0.4)
+		(layer "F.Cu")
+		(net 7)
+	)
+	(segment
+		(start 128.668629 66.3)
+		(end 160.7 66.3)
 		(width 0.4)
 		(layer "F.Cu")
@@
 	)
 	(segment
-		(start 107.5 72)
-		(end 107.5 70)
-		(width 0.4)
-		(layer "F.Cu")
-		(net 7)
-	)
-	(segment
-		(start 95.3 64.7)
-		(end 95.3 73)
+		(start 95.3 73)
+		(end 95.3 64.7)
+		(width 0.4)
+		(layer "F.Cu")
+		(net 7)
+	)
+	(segment
+		(start 105.5 74)
+		(end 96.3 74)
 		(width 0.4)
 		(layer "F.Cu")
@@
 		(width 0.4)
 		(layer "F.Cu")
+		(net 7)
+	)
+	(segment
+		(start 107.5 72)
+		(end 105.5 74)
+		(width 0.4)
+		(layer "F.Cu")
+		(net 7)
+	)
+	(segment
+		(start 96.3 74)
+		(end 95.3 73)
+		(width 0.4)
+		(layer "F.Cu")

Commit message: V2.1.7 - Première vérification
Parts:
- added REF**: MountingHole_3.2mm_M3, MountingHole:MountingHole_3.2mm_M3, F.Cu at (104.0, 88.5)
- added REF**: MountingHole_3.2mm_M3, MountingHole:MountingHole_3.2mm_M3, F.Cu at (184.0, 88.5)
- moved R10 0.50 mm to (117.7, 70.5)
- moved R9 0.50 mm to (117.6, 66.5)
Routing:
- net GND: track 0.00 -> 23.3 mm, vias 0 -> 1
- net /D0: track 229.7 -> 226.3 mm
- net Net-(U5-A): track 5.21 -> 5.99 mm
Other:
- board text added: "POP"
- board text added: "POR"
- board text added: "TP6"
